Commit message: changes for 4-wheel implementation

File: urdf/kangaroo_diff_drive_revolute.xacro (robot description, xacro)
@@ -32,10 +32,10 @@
              </visual>
            </link>
-           <joint type="continuous" name="${prefix}_motor_joint">
+           <joint type="revolute" name="${prefix}_motor_joint">
              <origin xyz="${reflect_fr*length/2} ${reflect_lr*axle_width/2} 0" rpy="0 0 0"/>
              <child link="${prefix}_wheel"/>
              <parent link="base_link"/>
              <axis xyz="0 1 0"/>
-             <limit effort="100" velocity="100.0" />
+             <limit effort="100" velocity="100.0"  lower="-5000" upper="5000" />
            </joint>
       </xacro:macro>
