Commit message: Updated dimensions

File: urdf/kangaroo_diff_drive.xacro (robot description, xacro)
@@ -4,7 +4,7 @@
   <xacro:property name="PI" value="3.1415926535897931"/>
   <xacro:property name = "chassis_width" value = "0.3"/>
-  <xacro:property name = "axle_width" value = "0.46"/>
-  <xacro:property name = "length" value = "0.6"/>
-  <xacro:property name = "wheel_t" value = "0.03"/>
+  <xacro:property name = "axle_width" value = "0.49"/>
+  <xacro:property name = "length" value = "0.57"/>
+  <xacro:property name = "wheel_t" value = "0.01"/>
   <xacro:property name = "wheel_r" value = "0.2"/>
   <!-- Base Link -->
